Commit message: modify parameters AMCL

File: catkin_ws/src/navigation/mybot_description/urdf/mybot.xacro (robot description, xacro)
@@ -177,5 +177,5 @@
   <!-- Hokuyo joint -->
   <joint name="hokuyo_joint" type="fixed">
-    <origin xyz="-0.13 0.0 0.35" rpy="0 0 0"/>
+    <origin xyz="0.13 0.0 0.35" rpy="0 0 0"/>
     <parent link="base_link"/>
     <axis xyz="0 1 0" />
